File: Hardware/we816mark2.kicad_pcb (KiCad board)
At the start: 2 copper layers, 360.1 x 141.4 mm, 146 parts, among them J1 AudioJack3, J10 DB9_Male, J11 DE15_Receptacle_HighDensity, J2 TTL Serial, J3 KEYBOARD, J4 IEC PORT, J5 CASELEDS, J6 INTERRUPT SELECT, J7 expansion port, J9 DB9_Male, K1 1&2 FOR SMALL ROM 2&3 FOR LAR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, K2 USE FOR 512K SRAM OR 128K SRAM, K3 1&2 FOR 27C256, 2&3 FOR 29C256, K4 VCC TOL 0, P1 SERIAL, P2 CHAN_MIX, P3 POWER, P4 RESET, P5 CLK_CPU, U1 W65C22NxP, U10 74AC04, U11 658C16, U12 GAL16V8, U13 GAL20V8, U14 GAL16V8, U15 16550, U17 MAX232, U2 7406, U20 74LS245, U21 74LS244, U22 74LS245, U23 74LS245, U24 74LS245, U25 AY-3-8910, U26 SRAM_512KO, U28 27C256, U29 27C512, U3 74LS06N, U30 74AC373, U31 74AC245, U32 74LVC245, U33 74LVC245, U34 74LVC245, U35 LM3940, U36 Pico, U37 DS1233, U4 74LS14, U5 W65C22NxP, U6 GAL16V8, U8 74LS175, U9 DS1210, X2 CXO_DIP8, X3 CRYSTAL 32.768 KHz

Commit message: pcb work
Parts:
- K1: value 1&2 FOR SMALL ROM 2&3 FOR LARGE ROM -> 1&2 FOR SMALL ROM, 2&3 FOR LARGE ROM
- P3: footprint TerminalBlock_RND:TerminalBlock_RND_205-00003_1x04_P5.00mm_Horizontal -> TerminalBlock_RND:TerminalBlock_RND_205-00001_1x02_P5.00mm_Horizontal
- moved C19 66.9 mm to (297.1, 146.1)
- moved JP2 57.5 mm to (221.0, 112.4)
- moved JP1 48.3 mm to (229.2, 124.5)
- moved R7 47.1 mm to (175.3, 175.9)
- moved C37 46.4 mm to (175.9, 137.8)
- moved R6 40.6 mm to (184.8, 181.0), turned to 180 degrees
- moved C21 35.1 mm to (123.2, 117.5)
- moved R5 34.3 mm to (184.8, 175.9), turned to 180 degrees
- moved U34 33.8 mm to (131.5, 124.5)
- moved C5 26.2 mm to (132.8, 120.0)
- moved C36 23.1 mm to (175.9, 130.2)
- moved R15 11.3 mm to (300.4, 205.1), turned to 0 degrees
- moved P3 7.32 mm to (47.7, 203.7)
- moved C9 4.45 mm to (353.7, 142.9)
- moved K3 4.11 mm to (290.2, 141.6)
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Routing:
- net GND: track 0.00 -> 2039.7 mm, vias 0 -> 29
- net VCC: track 0.00 -> 1636.7 mm, vias 0 -> 24
- net CLK_CPU: track 0.00 -> 625.0 mm, vias 0 -> 6
- net D1: track 0.00 -> 586.6 mm, vias 0 -> 8
- net A0: track 0.00 -> 584.7 mm, vias 0 -> 6
- net A1: track 0.00 -> 565.2 mm, vias 0 -> 7
- net A4: track 0.00 -> 563.4 mm, vias 0 -> 5
- net RW: track 0.00 -> 554.8 mm, vias 0 -> 4
- net A7: track 0.00 -> 549.5 mm, vias 0 -> 4
- net A3: track 0.00 -> 544.2 mm, vias 0 -> 10
- net D3: track 0.00 -> 534.5 mm, vias 0 -> 6
- net A2: track 0.00 -> 522.8 mm, vias 0 -> 6
- net D2: track 0.00 -> 521.8 mm, vias 0 -> 5
- net A5: track 0.00 -> 519.0 mm, vias 0 -> 7
- net D0: track 0.00 -> 516.7 mm, vias 0 -> 9
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- added copper zone on B.Cu, net GND
- added copper zone on F.Cu, net GND
Other:
- board text added: "+5V"
- board text added: "GND"

Commit message: graphics work
Parts:
- added U16: GAL16V8, Package_DIP:DIP-20_W7.62mm_Socket_LongPads, F.Cu at (168.7, 146.3)
- U1, U11, U5: footprint Package_DIP:DIP-40_W15.24mm_Socket -> Package_DIP:DIP-40_W15.24mm_Socket_LongPads
- U13: value GAL20V8 -> ATF22V10
- U15, U25: footprint Package_DIP:DIP-40_W15.24mm -> Package_DIP:DIP-40_W15.24mm_Socket_LongPads
- U2, U3: footprint Package_DIP:DIP-14_W7.62mm_Socket -> Package_DIP:DIP-14_W7.62mm_Socket_LongPads
- U26: footprint Package_DIP:DIP-32_W15.24mm -> Package_DIP:DIP-32_W15.24mm_Socket_LongPads
- U28, U29: footprint Package_DIP:DIP-28_W15.24mm -> Package_DIP:DIP-28_W15.24mm_Socket_LongPads
- U7: value ~ -> RP5C01
- U9: footprint Package_DIP:DIP-8_W7.62mm -> Package_DIP:DIP-8_W7.62mm_Socket_LongPads
- moved C14 145.6 mm to (225.5, 144.8)
- moved U13 76.9 mm to (212.9, 149.4)
- moved C4 24.4 mm to (171.7, 139.7)
Connections:
- J2 pad 1: VCC -> GND
- J2 pad 2: SIN_TTL -> RTS_TTL
- J2 pad 3: CTS_TTL -> VCC
- J2 pad 4: SOUT_TTL -> SIN_TTL
- J2 pad 5: RTS_TTL -> SOUT_TTL
- J2 pad 6: GND -> CTS_TTL
- U6 pad 18: unconnected-(U6-IO2-Pad18) -> VIDEO_WS
Routing:
- net GND: track 2039.7 -> 0.00 mm, vias 29 -> 0
- net VCC: track 1636.7 -> 0.00 mm, vias 24 -> 0
- net CLK_CPU: track 625.0 -> 0.00 mm, vias 6 -> 0
- net D1: track 586.6 -> 0.00 mm, vias 8 -> 0
- net A0: track 584.7 -> 0.00 mm, vias 6 -> 0
- net A1: track 565.2 -> 0.00 mm, vias 7 -> 0
- net A4: track 563.4 -> 0.00 mm, vias 5 -> 0
- net RW: track 554.8 -> 0.00 mm, vias 4 -> 0
- net A7: track 549.5 -> 0.00 mm, vias 4 -> 0
- net A3: track 544.2 -> 0.00 mm, vias 10 -> 0
- net D3: track 534.5 -> 0.00 mm, vias 6 -> 0
- net A2: track 522.8 -> 0.00 mm, vias 6 -> 0
- net D2: track 521.8 -> 0.00 mm, vias 5 -> 0
- net A5: track 519.0 -> 0.00 mm, vias 7 -> 0
- net D0: track 516.7 -> 0.00 mm, vias 9 -> 0
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- removed copper zone on B.Cu, net GND
- removed copper zone on F.Cu, net GND
Other:
- board text added: "65C816 PERSONAL COMPUTER MARK2 DAN WERNER - 8/11/2024 - V0.9"
- board text removed: "65C816 PERSONAL COMPUTER MARK2 DAN WERNER - 7/16/2024 - V.08"

Commit message: BASIC work
Parts:
- removed K1: 1&2 FOR SMALL ROM, 2&3 FOR LARGE ROM, Connector_PinHeader_2.54mm:PinHeader_1x03_P2.54mm_Vertical
Connections:
- U13 pad 20: Net-(K1-Pin_2) -> unconnected-(U13-I020-Pad20)
Routing:
- net GND: track 0.00 -> 1941.0 mm
- net VCC: track 0.00 -> 1619.0 mm, vias 0 -> 1
- net CLK_CPU: track 0.00 -> 583.7 mm, vias 0 -> 8
- net RW: track 0.00 -> 566.6 mm, vias 0 -> 2
- net A1: track 0.00 -> 560.1 mm, vias 0 -> 2
- net A0: track 0.00 -> 544.6 mm, vias 0 -> 3
- net A4: track 0.00 -> 531.4 mm, vias 0 -> 3
- net A6: track 0.00 -> 523.2 mm, vias 0 -> 4
- net D2: track 0.00 -> 514.4 mm, vias 0 -> 2
- net A2: track 0.00 -> 512.6 mm, vias 0 -> 2
- net D1: track 0.00 -> 510.5 mm, vias 0 -> 4
- net A7: track 0.00 -> 500.9 mm, vias 0 -> 2
- net D5: track 0.00 -> 496.7 mm, vias 0 -> 3
- net D4: track 0.00 -> 492.2 mm, vias 0 -> 1
- net A5: track 0.00 -> 484.9 mm, vias 0 -> 3
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- added copper zone on B.Cu, net GND
- added copper zone on F.Cu, net GND

Commit message: BASIC graphics work
Parts:
- added X1: CXO_DIP14, Oscillator:Oscillator_DIP-14, F.Cu at (149.0, 117.0)
- added X4: CXO_DIP14, Oscillator:Oscillator_DIP-14, F.Cu at (239.0, 117.0)
- J3: value KEYBOARD -> Keyboard
- J7: value expansion port -> Expansion Port
- moved J7 13.1 mm to (364.7, 77.7)
- moved P5 8.71 mm to (239.0, 117.0), turned to 0 degrees
- moved X2 7.62 mm to (149.0, 117.0), turned to 0 degrees
- moved J3 5.61 mm to (84.3, 141.7)
- moved C8 0.13 mm to (150.3, 105.2)
Connections:
- J3 pad 10: KB_GRAPH_LED -> ROWD
- J3 pad 11: KB_CAPS_LED -> COLUMN5
- J3 pad 12: ROWD -> KB_CAPS_LED
- J3 pad 13: ROWC -> COLUMN6
- J3 pad 14: ROWB -> KB_GRAPH_LED
- J3 pad 15: ROWA -> COLUMN7
- J3 pad 16: VCC -> GND
- J3 pad 2: COLUMN1 -> VCC
- J3 pad 3: COLUMN2 -> COLUMN1
- J3 pad 4: COLUMN3 -> ROWA
- J3 pad 5: COLUMN4 -> COLUMN2
- J3 pad 6: COLUMN5 -> ROWB
- J3 pad 7: COLUMN6 -> COLUMN3
- J3 pad 8: COLUMN7 -> ROWC
- J3 pad 9: GND -> COLUMN4
Routing:
- net GND: track 1941.0 -> 0.00 mm
- net VCC: track 1619.0 -> 0.00 mm, vias 1 -> 0
- net CLK_CPU: track 583.7 -> 0.00 mm, vias 8 -> 0
- net RW: track 566.6 -> 0.00 mm, vias 2 -> 0
- net A1: track 560.1 -> 0.00 mm, vias 2 -> 0
- net A0: track 544.6 -> 0.00 mm, vias 3 -> 0
- net A4: track 531.4 -> 0.00 mm, vias 3 -> 0
- net A6: track 523.2 -> 0.00 mm, vias 4 -> 0
- net D2: track 514.4 -> 0.00 mm, vias 2 -> 0
- net A2: track 512.6 -> 0.00 mm, vias 2 -> 0
- net D1: track 510.5 -> 0.00 mm, vias 4 -> 0
- net A7: track 500.9 -> 0.00 mm, vias 2 -> 0
- net D5: track 496.7 -> 0.00 mm, vias 3 -> 0
- net D4: track 492.2 -> 0.00 mm, vias 1 -> 0
- net A5: track 484.9 -> 0.00 mm, vias 3 -> 0
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- removed copper zone on B.Cu, net GND
- removed copper zone on F.Cu, net GND

Commit message: add plot commands to BASIC
Routing:
- net GND: track 0.00 -> 1946.5 mm, vias 0 -> 1
- net VCC: track 0.00 -> 1580.0 mm, vias 0 -> 1
- net A4: track 0.00 -> 605.7 mm, vias 0 -> 2
- net A1: track 0.00 -> 594.6 mm, vias 0 -> 5
- net CLK_CPU: track 0.00 -> 570.1 mm, vias 0 -> 4
- net RW: track 0.00 -> 561.8 mm, vias 0 -> 5
- net A2: track 0.00 -> 555.3 mm, vias 0 -> 5
- net D3: track 0.00 -> 547.8 mm, vias 0 -> 4
- net A0: track 0.00 -> 539.4 mm, vias 0 -> 3
- net A3: track 0.00 -> 536.3 mm, vias 0 -> 5
- net RESET: track 0.00 -> 527.4 mm, vias 0 -> 8
- net P2_L: track 0.00 -> 515.4 mm
- net A7: track 0.00 -> 513.0 mm, vias 0 -> 3
- net D4: track 0.00 -> 505.0 mm, vias 0 -> 3
- net D1: track 0.00 -> 504.4 mm, vias 0 -> 5
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- added copper zone on B.Cu, net GND
- added copper zone on F.Cu, net GND
Other:
- rule pad_to_mask_clearance: 0.254 -> 0

Commit message: rtc updates
Parts:
- removed BT1: Battery_Cell, CUSTOMLibrary:Battery_Holder_Coin_2032_BS-7_FIXED
- removed C34: 30 pF, Capacitor_THT:CP_Radial_D4.0mm_P2.00mm
- removed C36, C37: 33 pF, Capacitor_THT:C_Rect_L7.0mm_W2.0mm_P5.00mm
- removed JP1, JP2: BYPASS, Connector_PinHeader_2.54mm:PinHeader_1x02_P2.54mm_Vertical
- removed K4: VCC TOL 0, Connector_PinHeader_2.54mm:PinHeader_1x03_P2.54mm_Vertical
- removed R1, R2, R3: 100kΩ, Resistor_THT:R_Axial_DIN0204_L3.6mm_D1.6mm_P5.08mm_Horizontal
- removed U7: RP5C01, Package_DIP:DIP-18_W7.62mm_Socket_LongPads
- removed U8: 74LS175, Package_DIP:DIP-16_W7.62mm_Socket_LongPads
- removed U9: DS1210, Package_DIP:DIP-8_W7.62mm_Socket_LongPads
- added BT2: Battery_Cell, CUSTOMLibrary:Battery_Holder_Coin_2032_BS-7_FIXED, F.Cu at (152.9, 83.8)
- added U19: DS1501WN, Package_DIP:DIP-28_W15.24mm_Socket_LongPads, F.Cu at (186.9, 122.9)
- U30: value 74AC373 -> 74ALS373
- U31: value 74AC245 -> 74ALS245
Connections:
- U12 pad 12: unconnected-(U12-IO8-Pad12) -> VDA
Routing:
- net GND: track 1946.5 -> 0.00 mm, vias 1 -> 0
- net VCC: track 1580.0 -> 0.00 mm, vias 1 -> 0
- net A4: track 605.7 -> 0.00 mm, vias 2 -> 0
- net A1: track 594.6 -> 0.00 mm, vias 5 -> 0
- net CLK_CPU: track 570.1 -> 0.00 mm, vias 4 -> 0
- net RW: track 561.8 -> 0.00 mm, vias 5 -> 0
- net A2: track 555.3 -> 0.00 mm, vias 5 -> 0
- net D3: track 547.8 -> 0.00 mm, vias 4 -> 0
- net A0: track 539.4 -> 0.00 mm, vias 3 -> 0
- net A3: track 536.3 -> 0.00 mm, vias 5 -> 0
- net RESET: track 527.4 -> 0.00 mm, vias 8 -> 0
- net P2_L: track 515.4 -> 0.00 mm
- net A7: track 513.0 -> 0.00 mm, vias 3 -> 0
- net D4: track 505.0 -> 0.00 mm, vias 3 -> 0
- net D1: track 504.4 -> 0.00 mm, vias 5 -> 0
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- removed copper zone on B.Cu, net GND
- removed copper zone on F.Cu, net GND
Other:
- board text added: "65C816 PERSONAL COMPUTER MARK2 DAN WERNER - 9/7/2024 - V0.9"
- board text removed: "65C816 PERSONAL COMPUTER MARK2 DAN WERNER - 8/11/2024 - V0.9"
