File: Hardware/we816mark2.kicad_pcb (KiCad board)
At the start: 2 copper layers, 360.1 x 141.4 mm, 137 parts, among them J1 AudioJack3, J10 DB9_Male, J11 DE15_Receptacle_HighDensity, J2 TTL Serial, J3 Keyboard, J4 IEC PORT, J5 CASELEDS, J6 INTERRUPT SELECT, J7 Expansion Port, J9 DB9_Male, K2 USE FOR 512K SRAM OR 128K SRAM, K3 1&2 FOR 27C256, 2&3 FOR 29C256, P1 SERIAL, P2 CHAN_MIX, P3 POWER, P4 RESET, P5 CLK_CPU, U1 W65C22NxP, U10 74AC04, U11 658C16, U12 GAL16V8, U13 ATF22V10, U14 GAL16V8, U15 16550, U16 GAL16V8, U17 MAX232, U19 DS1501WN, U2 7406, U20 74LS245, U21 74LS244, U22 74LS245, U23 74LS245, U24 74LS245, U25 AY-3-8910, U26 SRAM_512KO, U28 27C256, U29 27C512, U3 74LS06N, U30 74ALS373, U31 74ALS245, U32 74LVC245, U33 74LVC245, U34 74LVC245, U35 LM3940, U36 Pico, U37 DS1233, U4 74LS14, U5 W65C22NxP, U6 GAL16V8, X1 CXO_DIP14, X2 CXO_DIP8, X3 CRYSTAL 32.768 KHz, X4 CXO_DIP14

Commit message: PCB work
Routing:
- net GND: track 0.00 -> 1953.9 mm
- net VCC: track 0.00 -> 1566.8 mm, vias 0 -> 2
- net CLK_CPU: track 0.00 -> 584.8 mm, vias 0 -> 2
- net A0: track 0.00 -> 584.7 mm, vias 0 -> 3
- net RW: track 0.00 -> 568.1 mm, vias 0 -> 4
- net D3: track 0.00 -> 556.9 mm, vias 0 -> 4
- net D4: track 0.00 -> 550.8 mm, vias 0 -> 4
- net A1: track 0.00 -> 529.5 mm, vias 0 -> 4
- net P2_R: track 0.00 -> 517.2 mm
- net D7: track 0.00 -> 514.1 mm, vias 0 -> 4
- net D5: track 0.00 -> 512.4 mm, vias 0 -> 5
- net A2: track 0.00 -> 511.3 mm, vias 0 -> 5
- net P2_L: track 0.00 -> 499.4 mm
- net A3: track 0.00 -> 493.5 mm, vias 0 -> 4
- net A7: track 0.00 -> 492.2 mm, vias 0 -> 4
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- added copper zone on B.Cu, net GND
- added copper zone on F.Cu, net GND

Commit message: add basic RTC functions
Parts:
- removed U16: GAL16V8, Package_DIP:DIP-20_W7.62mm_Socket_LongPads
Connections:
- U12 pad 18: ~{RTC_AD_WR} -> unconnected-(U12-IO2-Pad18)
- U6 pad 18: VIDEO_WS -> unconnected-(U6-IO2-Pad18)
Routing:
- net VIDEO_WS: track 89.7 -> 0.00 mm, vias 2 -> 0
- net WAIT: track 195.7 -> 116.6 mm, vias 4 -> 2
- net VDA: track 175.9 -> 112.3 mm
- net CS_ROM: track 146.4 -> 88.0 mm, vias 1 -> 0
- net VPA: track 157.2 -> 110.9 mm
- net CLK_CPU: track 584.8 -> 539.3 mm
- net IO: track 156.4 -> 141.7 mm
- net RW: track 568.1 -> 565.5 mm, vias 4 -> 5
- net VCC: track 1566.8 -> 1565.9 mm
- net GND: vias 0 -> 2
Other:
- board text added: "65C816 PERSONAL COMPUTER MARK2 DAN WERNER - 9/15/2024 - V1"
- board text removed: "65C816 PERSONAL COMPUTER MARK2 DAN WERNER - 9/7/2024 - V0.9"
