File: Hardware/file5FFCADA1.kicad_sch (KiCad schematic)
At the start: 21 parts, among them K2 USE FOR 512K SRAM OR 128K SRAM, K3 1&2 FOR 27C256, 2&3 FOR 29C256, P3 POWER, P4 RESET, P5 CLK_CPU, U26 SRAM_512KO, U27 658C16, U28 27C256, U29 27C512, U3 74LS06N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

Commit message: mark 2 work
Parts:
- removed C48: 22 µF, Capacitor_THT:CP_Radial_D4.0mm_P2.00mm, symbol Device:C_Polarized_Small
- removed C50: 10 µF, Capacitor_THT:CP_Radial_D4.0mm_P2.00mm, symbol Device:C_Polarized_Small
- removed P4: RESET, Connector_PinHeader_2.54mm:PinHeader_1x02_P2.54mm_Vertical, symbol Connector:Conn_01x02_Male
- removed R16: 10Ω, Resistor_THT:R_Axial_DIN0204_L3.6mm_D1.6mm_P5.08mm_Horizontal, symbol Device:R_Small
- removed R17: 10KΩ, Resistor_THT:R_Axial_DIN0204_L3.6mm_D1.6mm_P5.08mm_Horizontal, symbol Device:R_Small
- removed R18: 1KΩ, Resistor_THT:R_Axial_DIN0204_L3.6mm_D1.6mm_P5.08mm_Horizontal, symbol Device:R_Small
- removed U27: 658C16, Package_DIP:DIP-40_W15.24mm_Socket, symbol CUSTOM_CPU:65C816
- removed U3: 74LS06N, Package_DIP:DIP-14_W7.62mm_Socket, symbol 74xx:74LS06N
- removed unit 3 of U4
- added C35: 22 µF, Capacitor_THT:CP_Radial_D4.0mm_P2.00mm, symbol Device:C_Polarized_Small
- added P4: RESET, Connector_PinHeader_2.54mm:PinHeader_1x02_P2.54mm_Vertical, symbol Connector:Conn_01x02_Pin
- added R4: 10Ω, Resistor_THT:R_Axial_DIN0204_L3.6mm_D1.6mm_P5.08mm_Horizontal, symbol Device:R_Small
- added U10: 74AC04, Package_DIP:DIP-14_W7.62mm_Socket_LongPads, symbol 74xx:74HC04
- added U11: 658C16, Package_DIP:DIP-40_W15.24mm_Socket, symbol RPi_pico:65C816
- added U37: DS1233, Package_TO_SOT_THT:TO-92L_HandSolder, symbol Connector_Generic:Conn_01x03
- K2, K3: symbol Connector:Conn_01x03_Male -> Connector:Conn_01x03_Pin
- U30: value 74LS373 -> 74AC373
- U31: value 74LS245 -> 74AC245
Connections:
- net A0: now also U11.9 (A0)
- net A1: now also U11.10 (A1)
- net A10: now also U11.19 (A10)
- net A11: now also U11.20 (A11)
- net A12: now also U11.22 (A12)
- net A13: now also U11.23 (A13)
- net A14: now also U11.24 (A14)
- net A15: now also U11.25 (A15)
- net A2: now also U11.11 (A2)
- net A3: now also U11.12 (A3)
- net A4: now also U11.13 (A4)
- net A5: now also U11.14 (A5)
- net A6: now also U11.15 (A6)
- net A7: now also U11.16 (A7)
- net A8: now also U11.17 (A8)
- net A9: now also U11.18 (A9)
- net ABORT: now also U11.3 (~{ABORT})
- net AD0: now also U11.33 (AD0)
- net AD1: now also U11.32 (AD1)
- net AD2: now also U11.31 (AD2)
- net AD3: now also U11.30 (AD3)
- net AD4: now also U11.29 (AD4)
- net AD5: now also U11.28 (AD5)
- net AD6: now also U11.27 (AD6)
- net AD7: now also U11.26 (AD7)
- net BUSRQ: now also U11.36 (BE)
- net CLK_CPU: now also U10.1, U11.37 (CLK)
- net EMU: now also U11.35 (E)
- net GND: now also C35.2, P4.2 (Pin_2), U11.21 (GND), U37.1 (Pin_1)
- net INT: now also U11.4 (~{INT})
- net ML: now also U11.5 (~{ML})
- net NMI: now also U11.6 (~{NMI})
- net RESET: now also U4.3, R4.1, U11.40 (~{RESET}), U37.2 (Pin_2)
- net RW: now also U11.34 (R~{W})
- net VCC: now also C35.1, U11.8 (VCC), U37.3 (Pin_3)
- net VDA: now also U11.39 (VDA)
- net VP: now also U11.1 (~{VP})
- net VPA: now also U11.7 (VPA)
- net WAIT: now also U11.2 (RDY)
- net at U30.11 (LE), U31.19 (CE): now also U10.2
- new net: P4.1 (Pin_1), R4.2
Other:
- moved on the sheet: C49, K3, P5, U28, U29

Commit message: pcb work
Parts:
- P3: footprint TerminalBlock_RND:TerminalBlock_RND_205-00003_1x04_P5.00mm_Horizontal -> TerminalBlock_RND:TerminalBlock_RND_205-00001_1x02_P5.00mm_Horizontal
Other:
- title: (none) -> WE65816 - MARK2
Changed lines of the file:
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@@
 (kicad_sch (version 20230121) (generator eeschema)
   (paper "B")
+  (title_block
+    (title "WE65816 - MARK2")
+    (rev "V0.80")
+  )
   (junction (at 261.62 27.94) (diameter 0) (color 0 0 0 0)
   )
@@
       (effects (font (size 1.27 1.27)))
     )
-    (property "Footprint" "TerminalBlock_RND:TerminalBlock_RND_205-00003_1x04_P5.00mm_Horizontal" (at 162.56 213.36 0)
-      (effects (font (size 1.27 1.27)) hide)
-    )
+    (property "Footprint" "TerminalBlock_RND:TerminalBlock_RND_205-00001_1x02_P5.00mm_Horizontal" (at 162.56 213.36 0)
+      (effects (font (size 1.27 1.27)) hide)
+    )

Commit message: initial pico firmware
Changed lines of the file:
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@@
   (title_block
     (title "WE65816 - MARK2")
-    (rev "V0.80")
+    (rev "V0.90")
   )
   (junction (at 261.62 27.94) (diameter 0) (color 0 0 0 0)
@@
   )
   (symbol (lib_id "power:PWR_FLAG") (at 172.72 218.44 0) (unit 1)
-    (in_bom yes) (on_board yes) (dnp no) (fields_autoplaced)
+    (in_bom yes) (on_board yes) (dnp no)
     (property "Reference" "#FLG01" (at 172.72 216.535 0)
       (effects (font (size 1.27 1.27)) hide)
     )
-    (property "Value" "PWR_FLAG" (at 172.72 214.63 0)
+    (property "Value" "PWR_FLAG" (at 172.72 212.09 0)
       (effects (font (size 1.27 1.27)))
     )

Commit message: graphics work
Parts:
- U11: footprint Package_DIP:DIP-40_W15.24mm_Socket -> Package_DIP:DIP-40_W15.24mm_Socket_LongPads
- U26: footprint Package_DIP:DIP-32_W15.24mm -> Package_DIP:DIP-32_W15.24mm_Socket_LongPads
- U28, U29: footprint Package_DIP:DIP-28_W15.24mm -> Package_DIP:DIP-28_W15.24mm_Socket_LongPads
Changed lines of the file:
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@@
   (title_block
     (title "WE65816 - MARK2")
+    (date "2024-08-11")
     (rev "V0.90")
   )
@@
       (effects (font (size 1.778 1.778)) (justify left))
     )
-    (property "Footprint" "Package_DIP:DIP-32_W15.24mm" (at 59.69 149.86 0)
+    (property "Footprint" "Package_DIP:DIP-32_W15.24mm_Socket_LongPads" (at 59.69 149.86 0)
       (effects (font (size 1.27 1.27)) hide)
     )
@@
       (effects (font (size 1.27 1.27)))
     )
-    (property "Footprint" "Package_DIP:DIP-28_W15.24mm" (at 161.29 95.25 0)
+    (property "Footprint" "Package_DIP:DIP-28_W15.24mm_Socket_LongPads" (at 161.29 95.25 0)
       (effects (font (size 1.27 1.27)) hide)
     )
@@
       (effects (font (size 1.27 1.27)))
     )
-    (property "Footprint" "Package_DIP:DIP-28_W15.24mm" (at 246.38 95.25 0)
+    (property "Footprint" "Package_DIP:DIP-28_W15.24mm_Socket_LongPads" (at 246.38 95.25 0)
       (effects (font (size 1.27 1.27)) hide)
     )
@@
       (effects (font (size 1.524 1.524)) (justify left))
     )
-    (property "Footprint" "Package_DIP:DIP-40_W15.24mm_Socket" (at 82.55 43.18 0)
-      (effects (font (size 1.27 1.27)) hide)
-    )
+    (property "Footprint" "Package_DIP:DIP-40_W15.24mm_Socket_LongPads" (at 82.55 43.18 0)
+      (effects (font (size 1.27 1.27)) hide)
+    )

Commit message: BASIC graphics work
Parts:
- added X1: CXO_DIP14, Oscillator:Oscillator_DIP-14, symbol Oscillator:CXO_DIP14
Connections:
- net CLK_CPU: now also X1.8 (OUT)
- net GND: now also X1.7 (GND)
- net VCC: now also X1.1 (EN), X1.14 (Vcc)
Changed lines of the file:
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@@
   (junction (at 261.62 27.94) (diameter 0) (color 0 0 0 0)
   )
+  (junction (at 257.81 54.61) (diameter 0) (color 0 0 0 0)
+  )
   (junction (at 254 27.94) (diameter 0) (color 0 0 0 0)
   )
@@
   (junction (at 332.74 74.93) (diameter 0) (color 0 0 0 0)
   )
+  (junction (at 246.38 35.56) (diameter 0) (color 0 0 0 0)
+  )
   (junction (at 167.64 218.44) (diameter 0) (color 0 0 0 0)
   )
@@
   )
   (junction (at 162.56 232.41) (diameter 0) (color 0 0 0 0)
+  )
+  (junction (at 254 46.99) (diameter 0) (color 0 0 0 0)
   )
   (no_connect (at 64.77 72.39))
@@
     (stroke (width 0) (type default))
   )
+  (wire (pts (xy 246.38 35.56) (xy 241.3 35.56))
+    (stroke (width 0) (type default))
+  )
   (wire (pts (xy 374.65 57.15) (xy 377.19 57.15))
     (stroke (width 0) (type default))
@@
     (stroke (width 0) (type default))
   )
+  (wire (pts (xy 254 46.99) (xy 254 48.26))
+    (stroke (width 0) (type default))
+  )
   (wire (pts (xy 72.39 165.1) (xy 74.93 165.1))
     (stroke (width 0) (type default))
@@
     (stroke (width 0) (type default))
   )
+  (wire (pts (xy 250.19 62.23) (xy 250.19 46.99))
+    (stroke (width 0) (type default))
+  )
   (wire (pts (xy 62.23 100.33) (xy 64.77 100.33))
     (stroke (width 0) (type default))
@@
     (stroke (width 0) (type default))
   )
+  (wire (pts (xy 241.3 35.56) (xy 241.3 54.61))
+    (stroke (width 0) (type default))
+  )
   (wire (pts (xy 349.25 64.77) (xy 349.25 72.39))
     (stroke (width 0) (type default))
@@
     (stroke (width 0) (type default))
   )
+  (wire (pts (xy 265.43 46.99) (xy 267.97 46.99))
+    (stroke (width 0) (type default))
+  )
   (wire (pts (xy 161.29 123.19) (xy 161.29 125.73))
     (stroke (width 0) (type default))
@@
     (stroke (width 0) (type default))
   )
+  (wire (pts (xy 257.81 54.61) (xy 260.35 54.61))
+    (stroke (width 0) (type default))
+  )
   (wire (pts (xy 148.59 90.17) (xy 151.13 90.17))
     (stroke (width 0) (type default))
@@
     (stroke (width 0) (type default))
   )
+  (wire (pts (xy 246.38 35.56) (xy 246.38 27.94))
+    (stroke (width 0) (type default))
+  )
   (wire (pts (xy 205.74 125.73) (xy 190.5 125.73))
     (stroke (width 0) (type default))
@@
     (stroke (width 0) (type default))
   )
+  (wire (pts (xy 275.59 54.61) (xy 279.4 54.61))
+    (stroke (width 0) (type default))
+  )
   (wire (pts (xy 86.36 190.5) (xy 101.6 190.5))
     (stroke (width 0) (type default))
@@
     (stroke (width 0) (type default))
   )
-  (wire (pts (xy 254 45.72) (xy 254 48.26))
+  (wire (pts (xy 254 45.72) (xy 254 46.99))
     (stroke (width 0) (type default))
   )
@@
     (stroke (width 0) (type default))
   )
+  (wire (pts (xy 241.3 54.61) (xy 257.81 54.61))
+    (stroke (width 0) (type default))
+  )
   (wire (pts (xy 171.45 80.01) (xy 173.99 80.01))
     (stroke (width 0) (type default))
@@
     (stroke (width 0) (type default))
   )
+  (wire (pts (xy 257.81 54.61) (xy 257.81 48.26))
+    (stroke (width 0) (type default))
+  )
   (wire (pts (xy 72.39 175.26) (xy 74.93 175.26))
     (stroke (width 0) (type default))
@@
     (stroke (width 0) (type default))
   )
+  (wire (pts (xy 250.19 46.99) (xy 254 46.99))
+    (stroke (width 0) (type default))
+  )
   (wire (pts (xy 220.98 224.79) (xy 220.98 231.14))
     (stroke (width 0) (type default))
@@
     (stroke (width 0) (type default))
   )
-  (wire (pts (xy 246.38 38.1) (xy 246.38 27.94))
+  (wire (pts (xy 246.38 38.1) (xy 246.38 35.56))
     (stroke (width 0) (type default))
   )
@@
     (stroke (width 0) (type default))
   )
+  (wire (pts (xy 257.81 48.26) (xy 265.43 48.26))
+    (stroke (width 0) (type default))
+  )
+  (wire (pts (xy 265.43 48.26) (xy 265.43 46.99))
+    (stroke (width 0) (type default))
+  )
   (wire (pts (xy 171.45 107.95) (xy 173.99 107.95))
     (stroke (width 0) (type default))
@@
   )
   (wire (pts (xy 347.98 57.15) (xy 349.25 57.15))
+    (stroke (width 0) (type default))
+  )
+  (wire (pts (xy 267.97 62.23) (xy 250.19 62.23))
     (stroke (width 0) (type default))
   )
@@
     (effects (font (size 1.524 1.524)) (justify left))
     (property "Intersheetrefs" "${INTERSHEET_REFS}" (at -12.7 5.08 0)
+      (effects (font (size 1.27 1.27)) hide)
+    )
+  )
+  (global_label "CLK_CPU" (shape input) (at 279.4 54.61 0) (fields_autoplaced)
+    (effects (font (size 1.524 1.524)) (justify left))
+    (property "Intersheetrefs" "${INTERSHEET_REFS}" (at 62.23 -25.4 0)
       (effects (font (size 1.27 1.27)) hide)
     )
@@
         )
       )
+    )
+  )
+  (symbol (lib_id "Oscillator:CXO_DIP14") (at 267.97 54.61 0) (unit 1)
+    (in_bom yes) (on_board yes) (dnp no)
+    (property "Reference" "X1" (at 279.4 51.4859 0)
+      (effects (font (size 1.27 1.27)))
+    )
+    (property "Value" "CXO_DIP14" (at 274.32 46.99 0)
+      (effects (font (size 1.27 1.27)))
+    )
+    (property "Footprint" "Oscillator:Oscillator_DIP-14" (at 279.4 63.5 0)
+      (effects (font (size 1.27 1.27)) hide)
+    )
+    (property "Datasheet" "http://cdn-reichelt.de/documents/datenblatt/B400/OSZI.pdf" (at 265.43 54.61 0)
+      (effects (font (size 1.27 1.27)) hide)
+    )
+    (pin "1")
+    (pin "14")
+    (pin "7")
+    (pin "8")
+    (instances
+      (project "we816mark2"
+        (path "/ca9b74ce-0dee-401c-9544-f599f4cf538d/00000000-0000-0000-0000-00005ffce1f8"
+          (reference "X1") (unit 1)
+        )
+        (path "/ca9b74ce-0dee-401c-9544-f599f4cf538d/00000000-0000-0000-0000-00005ffcada2"
+          (reference "X4") (unit 1)
+        )
+      )

Commit message: rtc updates
Parts:
- U30: value 74AC373 -> 74ALS373
- U31: value 74AC245 -> 74ALS245
Changed lines of the file:
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@@
   (title_block
     (title "WE65816 - MARK2")
-    (date "2024-08-11")
+    (date "2024-09-07")
     (rev "V0.90")
   )
@@
       (effects (font (size 1.27 1.27)))
     )
-    (property "Value" "74AC373" (at 363.22 60.96 0)
+    (property "Value" "74ALS373" (at 363.22 60.96 0)
       (effects (font (size 1.27 1.27)))
     )
@@
       (effects (font (size 1.27 1.27)) (justify left bottom))
     )
-    (property "Value" "74AC245" (at 359.41 114.3 0)
+    (property "Value" "74ALS245" (at 359.41 114.3 0)
       (effects (font (size 1.27 1.27)) (justify left top))
     )
