File: Hardware/file5FFCBF10.kicad_sch (KiCad schematic)
At the start: 20 parts, among them J1 Conn_01x02_Male, Q1 2N3904, U10 RAM_32KO, U11 74LS32, U5 74LS04, U6 TMS9918, U7 74LS574, U8 74LS574, U9 74LS574, X1 10.7 MHz

Commit message: mark 2 work
Parts:
- removed C34, C35: 33 pF, Capacitor_THT:C_Rect_L7.0mm_W2.0mm_P5.00mm, symbol Device:C_Small
- removed C36: 22 µF, Capacitor_THT:CP_Radial_D4.0mm_P2.00mm, symbol Device:C_Polarized_Small
- removed C37: 0.1 µF, Capacitor_THT:C_Rect_L7.0mm_W2.0mm_P5.00mm, symbol Device:C_Small
- removed C38: 220 µF, Capacitor_THT:CP_Radial_D4.0mm_P2.00mm, symbol Device:C_Polarized_Small
- removed J1: Conn_01x02_Male, homecomputer2:CUI_RCJ-041, symbol Connector:Conn_01x02_Male
- removed L1: INDUCTOR (BEAD), Resistor_THT:R_Axial_DIN0207_L6.3mm_D2.5mm_P10.16mm_Horizontal, symbol Device:L_Small
- removed Q1: 2N3904, Package_TO_SOT_THT:TO-92L_HandSolder, symbol Device:Q_NPN_EBC
- removed R1: 0Ω, Resistor_THT:R_Axial_DIN0204_L3.6mm_D1.6mm_P5.08mm_Horizontal, symbol Device:R_Small
- removed R2: 470Ω, Resistor_THT:R_Axial_DIN0204_L3.6mm_D1.6mm_P5.08mm_Horizontal, symbol Device:R_Small
- removed R3, R4: 75Ω, Resistor_THT:R_Axial_DIN0204_L3.6mm_D1.6mm_P5.08mm_Horizontal, symbol Device:R_Small
- removed U10: RAM_32KO, Package_DIP:DIP-28_W15.24mm, symbol Memory_RAM:CY62256-70PC
- removed U11: 74LS32, Package_DIP:DIP-14_W7.62mm_Socket, symbol 74xx:74LS32
- removed U5: 74LS04, Package_DIP:DIP-14_W7.62mm_Socket, symbol 74xx:74LS04
- removed U6: TMS9918, Package_DIP:DIP-40_W15.24mm_Socket_LongPads, symbol CUSTOM_CPU:TMS9918
- removed U7: 74LS574, Package_DIP:DIP-20_W7.62mm_Socket, symbol 74xx:74LS574
- removed U8, U9: 74LS574, Package_DIP:DIP-20_W7.62mm_Socket_LongPads, symbol 74xx:74LS574
- removed X1: 10.7 MHz, Crystal:Crystal_HC18-U_Vertical, symbol Device:Crystal
- added J11: DE15_Receptacle_HighDensity, Connector_Dsub:DSUB-15-HD_Female_Horizontal_P2.29x1.98mm_EdgePinOffset3.03mm_Housed_MountingHolesOffset4.94mm, symbol Connector:DE15_Receptacle_HighDensity
- added R17, R18, R19: 1KΩ, Resistor_THT:R_Axial_DIN0204_L3.6mm_D1.6mm_P5.08mm_Horizontal, symbol Device:R_Small
- added R20, R23, R26: 510, Resistor_THT:R_Axial_DIN0204_L3.6mm_D1.6mm_P5.08mm_Horizontal, symbol Device:R_Small
- added R21, R24, R27: 1K, Resistor_THT:R_Axial_DIN0204_L3.6mm_D1.6mm_P5.08mm_Horizontal, symbol Device:R_Small
- added R22, R25, R28: 2K, Resistor_THT:R_Axial_DIN0204_L3.6mm_D1.6mm_P5.08mm_Horizontal, symbol Device:R_Small
- added R29, R31: 47, Resistor_THT:R_Axial_DIN0204_L3.6mm_D1.6mm_P5.08mm_Horizontal, symbol Device:R_Small
- added RN1: 10K, Resistor_THT:R_Array_SIP6, symbol Device:R_Network05
- added U32, U33, U34: 74LVC245, Package_DIP:DIP-20_W7.62mm_Socket_LongPads, symbol 74xx:74LS245
- added U36: Pico, RPi:RPi_Pico_SMD_TH, symbol RPi_pico:Pico
Connections:
- net A0: now also U33.11 (B7)
- net CS_VDP: now also R18.1
- net D0: now also U32.11 (B7)
- net D1: now also U32.12 (B6)
- net D2: now also U32.13 (B5)
- net D3: now also U32.14 (B4)
- net D4: now also U32.15 (B3)
- net D5: now also U32.16 (B2)
- net D6: now also U32.17 (B1)
- net D7: now also U32.18 (B0)
- net GND: now also J11.10, J11.5, J11.6, J11.7, J11.8, U32.10 (GND), U33.1 (A->B), U33.10 (GND), U34.1 (A->B), U34.10 (GND), U36.13 (GND), U36.18 (GND), U36.3 (GND), U36.8 (GND)
- new net: J11.14, R31.1
- new net: J11.2, R23.2, R24.2, R25.2
- new net: J11.13, R29.1
- new net: J11.1, R20.2, R21.2, R22.2
- new net: J11.3, R26.2, R27.2, R28.2
- new net +3.3V: RN1.1 (common), U32.20 (VCC), U33.20 (VCC), U34.20 (VCC), U36.39 (VSYS)
- new net A1: U33.12 (B6)
- new net A10: U34.13 (B5)
- new net A11: U34.14 (B4)
- new net A12: U34.15 (B3)
- new net A13: U34.16 (B2)
- new net A14: U34.17 (B1)
- new net A2: U33.13 (B5)
- new net A3: U33.14 (B4)
- new net A4: U33.15 (B3)
- new net A5: U33.16 (B2)
- new net A6: U33.17 (B1)
- new net A7: U33.18 (B0)
- new net A8: U34.11 (B7)
- new net A9: U34.12 (B6)
- new net CLK_CPU: R19.1
- new net HSYNC: R29.2, U36.34 (GPIO28_ADC2)
- new net RW: R17.1
- new net VADDR_HIGH: RN1.2 (R1), U34.19 (CE), U36.17 (GPIO13)
- new net VADDR_LOW: RN1.3 (R2), U33.19 (CE), U36.16 (GPIO12)
- new net VDATA: RN1.4 (R3), U32.19 (CE), U36.15 (GPIO11)
- new net VDATA_DIR: U32.1 (A->B), U36.14 (GPIO10)
- new net VDSEL: R18.2, RN1.5 (R4), U36.11 (GPIO8)
- new net VGAB1K: R27.1, U36.20 (GPIO15)
- new net VGAB2K: R28.1, U36.19 (GPIO14)
- new net VGAB500: R26.1, U36.21 (GPIO16)
- new net VGAG1L: R24.1, U36.24 (GPIO18)
- new net VGAG2K: R25.1, U36.22 (GPIO17)
- new net VGAG500: R23.1, U36.25 (GPIO19)
- new net VGAR1K: R21.1, U36.27 (GPIO21)
- new net VGAR2K: R22.1, U36.26 (GPIO20)
- new net VGAR500: R20.1, U36.29 (GPIO22)
- new net VIDEO_WINDOW: U34.18 (B0)
- new net VSYNC: R31.2, U36.32 (GPIO27_ADC1)
- new net V_CLK: R19.2, U36.31 (GPIO26_ADC0)
- new net V_DA0: U32.9 (A7), U33.9 (A7), U34.9 (A7), U36.1 (GPIO0)
- new net V_DA1: U32.8 (A6), U33.8 (A6), U34.8 (A6), U36.2 (GPIO1)
- new net V_DA2: U32.7 (A5), U33.7 (A5), U34.7 (A5), U36.4 (GPIO2)
- new net V_DA3: U32.6 (A4), U33.6 (A4), U34.6 (A4), U36.5 (GPIO3)
- new net V_DA4: U32.5 (A3), U33.5 (A3), U34.5 (A3), U36.6 (GPIO4)
- new net V_DA5: U32.4 (A2), U33.4 (A2), U34.4 (A2), U36.7 (GPIO5)
- new net V_DA6: U32.3 (A1), U33.3 (A1), U34.3 (A1), U36.9 (GPIO6)
- new net V_DA7: U32.2 (A0), U33.2 (A0), U34.2 (A0), U36.10 (GPIO7)
- new net V_RW: R17.2, U36.12 (GPIO9)
- no-connect marks 4 -> 18
Other:
- note added: "VIDEO"
- note removed: "C47 IS OPTIONAL. MOST MONITORS ARE CAPACITIVELY COUPLED ALREADY."
- note removed: "COMPOSITE VIDEO YELLOW RCA JACK"
- note removed: "SPRITE AND COLOR GRAPHICS VIDEO"

Commit message: pcb work
Other:
- title: (none) -> WE65816 - MARK2
Changed lines of the file:
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@@
 (kicad_sch (version 20230121) (generator eeschema)
   (paper "B")
+  (title_block
+    (title "WE65816 - MARK2")
+    (rev "V0.80")
+  )
   (junction (at 200.66 96.52) (diameter 0) (color 0 0 0 0)
   )
