File: Hardware/file5FFCD08B.kicad_sch (KiCad schematic)
At the start: 21 parts, among them J10 DB9_Male, J8 AudioJack3, J9 DB9_Male, P2 CHAN_MIX, U1 74LS393, U25 AY-3-8910

Commit message: mark 2 work
Parts:
- removed J8: AudioJack3, Connector_Audio:Jack_3.5mm_CUI_SJ1-3533NG_Horizontal_CircularHoles, symbol Connector:AudioJack3
- removed U1: 74LS393, Package_DIP:DIP-14_W7.62mm_Socket, symbol 74xx:74LS393
- added J1: AudioJack3, Connector_Audio:Jack_3.5mm_CUI_SJ1-3533NG_Horizontal_CircularHoles, symbol Connector_Audio:AudioJack3
- J10, J9: symbol Connector:DB9_Male -> Connector:DE9_Plug
Connections:
- net GND: now also J1.T
- net CLK_UART: now reaches U25.22 (CLOCK)
- net at C46.2: now also J1.S
- net at C47.2: now also J1.R
- no-connect marks 12 -> 9

Commit message: pcb work
Other:
- title: (none) -> WE65816 - MARK2
Changed lines of the file:
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@@
 (kicad_sch (version 20230121) (generator eeschema)
   (paper "B")
+  (title_block
+    (title "WE65816 - MARK2")
+    (rev "V0.80")
+  )
   (junction (at 248.92 124.46) (diameter 0) (color 0 0 0 0)
   )

Commit message: initial pico firmware
Changed lines of the file:
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@@
   (title_block
     (title "WE65816 - MARK2")
-    (rev "V0.80")
+    (rev "V0.90")
   )
   (junction (at 248.92 124.46) (diameter 0) (color 0 0 0 0)
@@
       (effects (font (size 1.524 1.524)))
     )
-    (property "Value" "AY-3-8910" (at 143.51 100.33 0)
+    (property "Value" "AY-3-8910" (at 139.7 128.27 0)
       (effects (font (size 1.524 1.524)))
     )

Commit message: graphics work
Parts:
- U25: footprint Package_DIP:DIP-40_W15.24mm -> Package_DIP:DIP-40_W15.24mm_Socket_LongPads
Changed lines of the file:
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@@
   (title_block
     (title "WE65816 - MARK2")
+    (date "2024-08-11")
     (rev "V0.90")
   )
@@
       (effects (font (size 1.524 1.524)))
     )
-    (property "Footprint" "Package_DIP:DIP-40_W15.24mm" (at 158.75 144.78 0)
-      (effects (font (size 1.27 1.27)) hide)
-    )
+    (property "Footprint" "Package_DIP:DIP-40_W15.24mm_Socket_LongPads" (at 158.75 144.78 0)
+      (effects (font (size 1.27 1.27)) hide)
+    )
