File: Hardware/file5FFCE1F7.kicad_sch (KiCad schematic)
At the start: 22 parts, among them J2 TTL Serial, J3 KEYBOARD, J4 IEC PORT, J5 CASELEDS, P1 SERIAL, U15 16550, U16 DS1302, U17 MAX232, U18 W65C22NxP, U19 W65C22NxP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

Commit message: mark 2 work
Parts:
- removed U16: DS1302, Package_DIP:DIP-8_W7.62mm, symbol Timer_RTC:DS1302+
- removed U18, U19: W65C22NxP, Package_DIP:DIP-40_W15.24mm_Socket, symbol CUSTOM_CPU:65C22
- added C21 (x2): 33 pF, Capacitor_THT:C_Rect_L7.0mm_W2.0mm_P5.00mm, symbol Device:C_Small
- added C34: 30 pF, Capacitor_THT:CP_Radial_D4.0mm_P2.00mm, symbol Device:C_Trim_Small
- added JP1, JP2: BYPASS, Connector_PinHeader_2.54mm:PinHeader_1x02_P2.54mm_Vertical, symbol Jumper:Jumper_2_Open
- added K4: VCC TOL 0, Connector_PinHeader_2.54mm:PinHeader_1x03_P2.54mm_Vertical, symbol Connector_Generic:Conn_01x03
- added R16 (x3): 100kΩ, Resistor_THT:R_Axial_DIN0204_L3.6mm_D1.6mm_P5.08mm_Horizontal, symbol Device:R_Small
- added U1, U5: W65C22NxP, Package_DIP:DIP-40_W15.24mm_Socket, symbol RPi_pico:65C22
- added U7: ~, Package_DIP:DIP-18_W7.62mm_Socket_LongPads, symbol RPi_pico:rp5c01
- added U8: 74LS175, Package_DIP:DIP-16_W7.62mm_Socket_LongPads, symbol 74xx:74LS175
- added U9: DS1210, Package_DIP:DIP-8_W7.62mm, symbol Power_Management:DS1210
- BT1: footprint homecomputer2:Battery_Holder_Coin_2032_BS-7_FIXED -> CUSTOMLibrary:Battery_Holder_Coin_2032_BS-7_FIXED
- J2: symbol Connector:Conn_01x06_Male -> Connector:Conn_01x06_Pin
- J4: footprint Connector:din6 -> CUSTOMLibrary:din6
- J5: symbol Connector:Conn_01x03_Male -> Connector:Conn_01x03_Pin
Connections:
- net A0: now also U1.38 (RS0), U5.38 (RS0)
- net A1: now also U1.37 (RS1), U5.37 (RS1)
- net A2: now also U1.36 (RS2), U5.36 (RS2)
- net A3: now also U1.35 (RS3), U5.35 (RS3)
- net CLK_CPU: now also U1.25 (CLK), U5.25 (CLK)
- net COLUMN0: now also U5.2 (PA0)
- net COLUMN1: now also U5.3 (PA1)
- net COLUMN2: now also U5.4 (PA2)
- net COLUMN3: now also U5.5 (PA3)
- net COLUMN4: now also U5.6 (PA4)
- net COLUMN5: now also U5.7 (PA5)
- net COLUMN6: now also U5.8 (PA6)
- net COLUMN7: now also U5.9 (PA7)
- net CS_VIA1: now also U1.23 (~{CS2})
- net CS_VIA2: now also U5.23 (~{CS2})
- net D0: now also U1.33 (D0), U5.33 (D0), U7.11 (D0), U8.4 (D0)
- net D1: now also U1.32 (D1), U5.32 (D1), U7.12 (D1), U8.5 (D1)
- net D2: now also U1.31 (D2), U5.31 (D2), U7.13 (D2), U8.12 (D2)
- net D3: now also U1.30 (D3), U5.30 (D3), U7.14 (D3), U8.13 (D3)
- net D4: now also U1.29 (D4), U5.29 (D4)
- net D5: now also U1.28 (D5), U5.28 (D5)
- net D6: now also U1.27 (D6), U5.27 (D6)
- net D7: now also U1.26 (D7), U5.26 (D7)
- net GND: now also C21.1, C21.2, C34.2, K4.3 (Pin_3), R16.2, U1.1 (VSS), U5.1 (VSS), U7.9 (GND), U8.8 (GND), U9.4 (GND); no longer BT1.2 (-)
- net KB_CAPS_LED: now also U5.14 (PB4)
- net KB_GRAPH_LED: now also U5.15 (PB5)
- net LED_1: now also U5.16 (PB6)
- net LED_2: now also U5.17 (PB7)
- net RD: now also U7.8 (~{RD})
- net RESET: now also U1.34 (~{RESET}), U5.34 (~{RESET}), U8.1 (~{Mr})
- net ROWA: now also U5.10 (PB0)
- net ROWB: now also U5.11 (PB1)
- net ROWC: now also U5.12 (PB2)
- net ROWD: now also U5.13 (PB3)
- net RW: now also U1.22 (R/~{W}), U5.22 (R/~{W})
- net SERATNOUT: now also U1.9 (PA7)
- net SERCLKIN: now also U1.2 (PA0)
- net SERCLKOUT: now also U5.39 (CA2)
- net SERDATAIN: now also U1.3 (PA1)
- net SERDATAOUT: now also U5.19 (CB2)
- net SERSRQ: now also U5.18 (CB1)
- net USERA_2: now also U1.4 (PA2)
- net USERA_3: now also U1.5 (PA3)
- net USERA_4: now also U1.6 (PA4)
- net USERB_0: now also U1.10 (PB0)
- net USERB_1: now also U1.11 (PB1)
- net USERB_2: now also U1.12 (PB2)
- net USERB_3: now also U1.13 (PB3)
- net USERB_4: now also U1.14 (PB4)
- net USERB_5: now also U1.15 (PB5)
- net USERB_6: now also U1.16 (PB6)
- net USERB_7: now also U1.17 (PB7)
- net USERCA_2: now also U1.39 (CA2), U7.15 (~{ALARM})
- net VCC: now also JP2.1 (A), R16.1, U1.20 (VCC), U1.24 (CS1), U5.20 (VCC), U5.24 (CS1), U8.16 (VCC), U9.8 (VCCI)
- net VIA1_INT: now also U1.21 (~{IRQ})
- net VIA2_INT: now also U5.21 (~{IRQ})
- net VRAM_BANK: now also U5.40 (CA1)
- net WR: now also U7.10 (~{WR})
- net at X3.1: now also C21.2, R16.2
- net at X3.2: now also C34.1, U7.16 (OSCIN)
- net at BT1.1 (+): now also U9.2 (VBAT1)
- new net: BT1.2 (-), U9.7 (VBAT2)
- new net: R16.1, U7.3 (ADJ)
- new net: C21.1, R16.1, U7.17 (OSCOUT)
- new net: R16.2, U7.2 (CS)
- new net: U7.4 (A0), U8.2 (Q0)
- new net: U7.5 (A1), U8.7 (Q1)
- new net: U7.6 (A2), U8.10 (Q2)
- new net: U7.7 (A3), U8.15 (Q3)
- new net: K4.2 (Pin_2), U9.3 (TOL)
- new net VCC_RTC: JP2.2 (B), K4.1 (Pin_1), U7.18 (VCC), U9.1 (VCCO)
- new net ~{RTC_AD_WR}: U8.9 (Cp)
- new net ~{RTC_CS_O}: JP1.2 (B), U7.1 (~{CS}), U9.6 (~{CEO})
- new net ~{RTC_CS}: JP1.1 (A), U9.5 (~{CE})
- no-connect marks 18 -> 24
Other:
- note added: "JP1 AND JP3 U2 DS1210 INSTALLED CLOSE BOTH TO BYPASS DEFAULT BOTH OPEN"
- note added: "NOTE: K1 VCC TOLERANCE 1-2 CLOSED 10% 2-3 CLOSED 5%"
- moved on the sheet: BT1, C39, C40, C41, C42, C43, U17, X3

Commit message: pcb work
Other:
- title: (none) -> WE65816 - MARK2
Changed lines of the file:
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@@
 (kicad_sch (version 20230121) (generator eeschema)
   (paper "B")
+  (title_block
+    (title "WE65816 - MARK2")
+    (rev "V0.80")
+  )
   (junction (at 367.03 41.91) (diameter 0) (color 0 0 0 0)
   )

Commit message: graphics work
Parts:
- U1, U5: footprint Package_DIP:DIP-40_W15.24mm_Socket -> Package_DIP:DIP-40_W15.24mm_Socket_LongPads
- U15: footprint Package_DIP:DIP-40_W15.24mm -> Package_DIP:DIP-40_W15.24mm_Socket_LongPads
- U2: footprint Package_DIP:DIP-14_W7.62mm_Socket -> Package_DIP:DIP-14_W7.62mm_Socket_LongPads
- U7: value ~ -> RP5C01
- U9: footprint Package_DIP:DIP-8_W7.62mm -> Package_DIP:DIP-8_W7.62mm_Socket_LongPads
Connections:
- net CTS_TTL: now also J2.6 (Pin_6); no longer J2.3 (Pin_3)
- net GND: now also J2.1 (Pin_1); no longer J2.6 (Pin_6)
- net RTS_TTL: now also J2.2 (Pin_2); no longer J2.5 (Pin_5)
- net SIN_TTL: now also J2.4 (Pin_4); no longer J2.2 (Pin_2)
- net SOUT_TTL: now also J2.5 (Pin_5); no longer J2.4 (Pin_4)
- net VCC: now also J2.3 (Pin_3); no longer J2.1 (Pin_1)
Other:
- note added: "TTL SERIAL TO USB CONNECTOR"
Changed lines of the file:
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@@
   (title_block
     (title "WE65816 - MARK2")
+    (date "2024-08-11")
     (rev "V0.90")
   )
@@
     (stroke (width 0) (type default))
   )
-  (wire (pts (xy 92.71 215.9) (xy 111.76 215.9))
-    (stroke (width 0) (type default))
-  )
   (wire (pts (xy 201.93 36.83) (xy 201.93 41.91))
     (stroke (width 0) (type default))
@@
     (stroke (width 0) (type default))
   )
-  (wire (pts (xy 92.71 203.2) (xy 111.76 203.2))
+  (wire (pts (xy 92.71 203.2) (xy 116.84 203.2))
     (stroke (width 0) (type default))
   )
@@
     (stroke (width 0) (type default))
   )
-  (wire (pts (xy 92.71 208.28) (xy 97.79 208.28))
+  (wire (pts (xy 92.71 208.28) (xy 113.03 208.28))
     (stroke (width 0) (type default))
   )
@@
     (stroke (width 0) (type default))
   )
+  (wire (pts (xy 92.71 215.9) (xy 97.79 215.9))
+    (stroke (width 0) (type default))
+  )
   (wire (pts (xy 63.5 208.28) (xy 67.31 208.28))
     (stroke (width 0) (type default))
@@
     (stroke (width 0) (type default))
   )
+  (text "TTL SERIAL TO \nUSB CONNECTOR" (at 85.09 224.79 0)
+    (effects (font (size 1.524 1.524)) (justify left bottom))
+  )
   (text "SERIAL IO" (at 67.31 97.79 0)
     (effects (font (size 1.524 1.524)) (justify left bottom))
@@
     )
   )
-  (global_label "SOUT_TTL" (shape input) (at 97.79 210.82 0) (fields_autoplaced)
+  (global_label "SOUT_TTL" (shape input) (at 97.79 213.36 0) (fields_autoplaced)
     (effects (font (size 1.524 1.524)) (justify left))
-    (property "Intersheetrefs" "${INTERSHEET_REFS}" (at 254 351.79 0)
+    (property "Intersheetrefs" "${INTERSHEET_REFS}" (at 254 354.33 0)
       (effects (font (size 1.27 1.27)) hide)
     )
@@
     )
   )
-  (global_label "SIN_TTL" (shape input) (at 97.79 205.74 0) (fields_autoplaced)
+  (global_label "SIN_TTL" (shape input) (at 97.79 210.82 0) (fields_autoplaced)
     (effects (font (size 1.524 1.524)) (justify left))
-    (property "Intersheetrefs" "${INTERSHEET_REFS}" (at 254 351.79 0)
+    (property "Intersheetrefs" "${INTERSHEET_REFS}" (at 254 356.87 0)
       (effects (font (size 1.27 1.27)) hide)
     )
@@
     )
   )
-  (global_label "RTS_TTL" (shape input) (at 97.79 213.36 0) (fields_autoplaced)
+  (global_label "RTS_TTL" (shape input) (at 97.79 205.74 0) (fields_autoplaced)
     (effects (font (size 1.524 1.524)) (justify left))
-    (property "Intersheetrefs" "${INTERSHEET_REFS}" (at 254 351.79 0)
+    (property "Intersheetrefs" "${INTERSHEET_REFS}" (at 254 344.17 0)
       (effects (font (size 1.27 1.27)) hide)
     )
@@
     )
   )
-  (global_label "CTS_TTL" (shape input) (at 97.79 208.28 0) (fields_autoplaced)
+  (global_label "CTS_TTL" (shape input) (at 97.79 215.9 0) (fields_autoplaced)
     (effects (font (size 1.524 1.524)) (justify left))
-    (property "Intersheetrefs" "${INTERSHEET_REFS}" (at 254 351.79 0)
+    (property "Intersheetrefs" "${INTERSHEET_REFS}" (at 254 359.41 0)
       (effects (font (size 1.27 1.27)) hide)
     )
@@
       (effects (font (size 1.778 1.778)))
     )
-    (property "Footprint" "Package_DIP:DIP-40_W15.24mm" (at 71.12 148.59 0)
+    (property "Footprint" "Package_DIP:DIP-40_W15.24mm_Socket_LongPads" (at 71.12 148.59 0)
       (effects (font (size 1.27 1.27) italic) hide)
     )
@@
       (effects (font (size 1.27 1.27)))
     )
-    (property "Footprint" "Package_DIP:DIP-14_W7.62mm_Socket" (at 354.33 24.13 0)
+    (property "Footprint" "Package_DIP:DIP-14_W7.62mm_Socket_LongPads" (at 354.33 24.13 0)
       (effects (font (size 1.27 1.27)) hide)
     )
@@
       (effects (font (size 1.27 1.27)))
     )
-    (property "Footprint" "Package_DIP:DIP-14_W7.62mm_Socket" (at 353.06 41.91 0)
+    (property "Footprint" "Package_DIP:DIP-14_W7.62mm_Socket_LongPads" (at 353.06 41.91 0)
       (effects (font (size 1.27 1.27)) hide)
     )
@@
       (effects (font (size 1.27 1.27)))
     )
-    (property "Footprint" "Package_DIP:DIP-14_W7.62mm_Socket" (at 353.06 59.69 0)
+    (property "Footprint" "Package_DIP:DIP-14_W7.62mm_Socket_LongPads" (at 353.06 59.69 0)
       (effects (font (size 1.27 1.27)) hide)
     )
@@
     )
   )
-  (symbol (lib_id "power:GND") (at 111.76 215.9 0) (unit 1)
+  (symbol (lib_id "power:GND") (at 116.84 203.2 0) (unit 1)
     (in_bom yes) (on_board yes) (dnp no)
-    (property "Reference" "#PWR038" (at 111.76 215.9 0)
+    (property "Reference" "#PWR038" (at 116.84 203.2 0)
       (effects (font (size 0.762 0.762)) hide)
     )
-    (property "Value" "GND" (at 111.76 217.678 0)
+    (property "Value" "GND" (at 116.84 204.978 0)
       (effects (font (size 0.762 0.762)) hide)
     )
-    (property "Footprint" "" (at 111.76 215.9 0)
+    (property "Footprint" "" (at 116.84 203.2 0)
       (effects (font (size 1.27 1.27)) hide)
     )
-    (property "Datasheet" "" (at 111.76 215.9 0)
+    (property "Datasheet" "" (at 116.84 203.2 0)
       (effects (font (size 1.27 1.27)) hide)
     )
@@
   )
   (symbol (lib_id "RPi_pico:rp5c01") (at 125.73 44.45 0) (unit 1)
-    (in_bom yes) (on_board yes) (dnp no) (fields_autoplaced)
+    (in_bom yes) (on_board yes) (dnp no)
     (property "Reference" "U7" (at 127.6859 30.48 0)
       (effects (font (size 1.27 1.27)) (justify left))
     )
-    (property "Value" "~" (at 125.73 44.45 0)
+    (property "Value" "RP5C01" (at 125.73 50.8 0)
       (effects (font (size 1.27 1.27)))
     )
@@
     )
   )
-  (symbol (lib_id "power:VCC") (at 111.76 203.2 0) (unit 1)
+  (symbol (lib_id "power:VCC") (at 113.03 208.28 0) (unit 1)
     (in_bom yes) (on_board yes) (dnp no)
-    (property "Reference" "#PWR037" (at 111.76 207.01 0)
+    (property "Reference" "#PWR037" (at 113.03 212.09 0)
       (effects (font (size 1.27 1.27)) hide)
     )
-    (property "Value" "VCC" (at 112.141 198.8058 0)
+    (property "Value" "VCC" (at 115.57 208.28 0)
       (effects (font (size 1.27 1.27)))
     )
-    (property "Footprint" "" (at 111.76 203.2 0)
+    (property "Footprint" "" (at 113.03 208.28 0)
       (effects (font (size 1.27 1.27)) hide)
     )
-    (property "Datasheet" "" (at 111.76 203.2 0)
+    (property "Datasheet" "" (at 113.03 208.28 0)
       (effects (font (size 1.27 1.27)) hide)
     )
@@
       (effects (font (size 1.27 1.27) bold italic) (justify left))
     )
-    (property "Footprint" "Package_DIP:DIP-40_W15.24mm_Socket" (at 312.42 125.73 0)
+    (property "Footprint" "Package_DIP:DIP-40_W15.24mm_Socket_LongPads" (at 312.42 125.73 0)
       (effects (font (size 1.27 1.27)) hide)
     )
@@
       (effects (font (size 1.27 1.27)))
     )
-    (property "Footprint" "Package_DIP:DIP-8_W7.62mm" (at 185.42 143.51 0)
+    (property "Footprint" "Package_DIP:DIP-8_W7.62mm_Socket_LongPads" (at 185.42 143.51 0)
       (effects (font (size 1.27 1.27)) hide)
     )
@@
       (effects (font (size 1.27 1.27) bold italic) (justify left))
     )
-    (property "Footprint" "Package_DIP:DIP-40_W15.24mm_Socket" (at 278.13 36.83 0)
+    (property "Footprint" "Package_DIP:DIP-40_W15.24mm_Socket_LongPads" (at 278.13 36.83 0)
       (effects (font (size 1.27 1.27)) hide)
     )

Commit message: BASIC graphics work
Parts:
- removed J3: KEYBOARD, Connector_PinHeader_2.54mm:PinHeader_2x08_P2.54mm_Vertical, symbol Connector_Generic:Conn_02x08_Counter_Clockwise
- added J3: Keyboard, Connector_PinHeader_2.54mm:PinHeader_2x08_P2.54mm_Vertical, symbol Connector_Generic:Conn_02x08_Odd_Even
- added X1: CXO_DIP14, Oscillator:Oscillator_DIP-14, symbol Oscillator:CXO_DIP14
Connections:
- net CLK_UART: now also X1.8 (OUT)
- net COLUMN0: now also J3.1 (Pin_1)
- net COLUMN1: now also J3.3 (Pin_3)
- net COLUMN2: now also J3.5 (Pin_5)
- net COLUMN3: now also J3.7 (Pin_7)
- net COLUMN4: now also J3.9 (Pin_9)
- net COLUMN5: now also J3.11 (Pin_11)
- net COLUMN6: now also J3.13 (Pin_13)
- net COLUMN7: now also J3.15 (Pin_15)
- net GND: now also J3.16 (Pin_16), X1.7 (GND)
- net KB_CAPS_LED: now also J3.12 (Pin_12)
- net KB_GRAPH_LED: now also J3.14 (Pin_14)
- net ROWA: now also J3.4 (Pin_4)
- net ROWB: now also J3.6 (Pin_6)
- net ROWC: now also J3.8 (Pin_8)
- net ROWD: now also J3.10 (Pin_10)
- net VCC: now also J3.2 (Pin_2), X1.1 (EN), X1.14 (Vcc)
Changed lines of the file:
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@@
   (junction (at 200.66 107.95) (diameter 0) (color 0 0 0 0)
   )
+  (junction (at 27.94 238.76) (diameter 0) (color 0 0 0 0)
+  )
   (junction (at 33.02 143.51) (diameter 0) (color 0 0 0 0)
   )
@@
   (junction (at 200.66 99.06) (diameter 0) (color 0 0 0 0)
   )
+  (junction (at 38.1 247.65) (diameter 0) (color 0 0 0 0)
+  )
   (junction (at 167.64 144.78) (diameter 0) (color 0 0 0 0)
   )
@@
   (junction (at 171.45 36.83) (diameter 0) (color 0 0 0 0)
   )
+  (junction (at 40.64 254) (diameter 0) (color 0 0 0 0)
+  )
   (junction (at 38.1 231.14) (diameter 0) (color 0 0 0 0)
   )
@@
     (stroke (width 0) (type default))
   )
+  (wire (pts (xy 41.91 254) (xy 40.64 254))
+    (stroke (width 0) (type default))
+  )
   (wire (pts (xy 165.1 39.37) (xy 165.1 50.8))
     (stroke (width 0) (type default))
@@
     (stroke (width 0) (type default))
   )
+  (wire (pts (xy 40.64 254) (xy 27.94 254))
+    (stroke (width 0) (type default))
+  )
   (wire (pts (xy 185.42 133.35) (xy 185.42 135.89))
     (stroke (width 0) (type default))
@@
     (stroke (width 0) (type default))
   )
-  (wire (pts (xy 38.1 246.38) (xy 38.1 248.92))
+  (wire (pts (xy 38.1 246.38) (xy 38.1 247.65))
     (stroke (width 0) (type default))
   )
@@
     (stroke (width 0) (type default))
   )
+  (wire (pts (xy 49.53 261.62) (xy 34.29 261.62))
+    (stroke (width 0) (type default))
+  )
   (wire (pts (xy 195.58 144.78) (xy 195.58 128.27))
     (stroke (width 0) (type default))
@@
     (stroke (width 0) (type default))
   )
+  (wire (pts (xy 57.15 254) (xy 59.69 254))
+    (stroke (width 0) (type default))
+  )
   (wire (pts (xy 171.45 187.96) (xy 171.45 186.69))
     (stroke (width 0) (type default))
@@
     (stroke (width 0) (type default))
   )
+  (wire (pts (xy 34.29 261.62) (xy 34.29 247.65))
+    (stroke (width 0) (type default))
+  )
   (wire (pts (xy 388.62 33.02) (xy 388.62 29.21))
     (stroke (width 0) (type default))
@@
     (stroke (width 0) (type default))
   )
+  (wire (pts (xy 27.94 254) (xy 27.94 238.76))
+    (stroke (width 0) (type default))
+  )
   (wire (pts (xy 365.76 19.05) (xy 367.03 19.05))
     (stroke (width 0) (type default))
@@
     (stroke (width 0) (type default))
   )
+  (wire (pts (xy 40.64 246.38) (xy 40.64 254))
+    (stroke (width 0) (type default))
+  )
   (wire (pts (xy 392.43 160.02) (xy 393.7 160.02))
     (stroke (width 0) (type default))
@@
     (stroke (width 0) (type default))
   )
+  (wire (pts (xy 34.29 247.65) (xy 38.1 247.65))
+    (stroke (width 0) (type default))
+  )
   (wire (pts (xy 41.91 168.91) (xy 45.72 168.91))
     (stroke (width 0) (type default))
@@
     (stroke (width 0) (type default))
   )
+  (wire (pts (xy 49.53 246.38) (xy 40.64 246.38))
+    (stroke (width 0) (type default))
+  )
   (wire (pts (xy 392.43 149.86) (xy 393.7 149.86))
     (stroke (width 0) (type default))
@@
     (stroke (width 0) (type default))
   )
+  (wire (pts (xy 38.1 247.65) (xy 38.1 248.92))
+    (stroke (width 0) (type default))
+  )
   (wire (pts (xy 290.83 71.12) (xy 297.18 71.12))
     (stroke (width 0) (type default))
@@
     )
   )
+  (global_label "CLK_UART" (shape input) (at 59.69 254 0) (fields_autoplaced)
+    (effects (font (size 1.524 1.524)) (justify left))
+    (property "Intersheetrefs" "${INTERSHEET_REFS}" (at -22.86 10.16 0)
+      (effects (font (size 1.27 1.27)) hide)
+    )
+  )
   (global_label "A2" (shape input) (at 261.62 58.42 180) (fields_autoplaced)
     (effects (font (size 1.524 1.524)) (justify right))
@@
     )
   )
-  (symbol (lib_id "Connector_Generic:Conn_02x08_Counter_Clockwise") (at 384.81 149.86 0) (unit 1)
-    (in_bom yes) (on_board yes) (dnp no)
-    (property "Reference" "J3" (at 386.08 136.7282 0)
-      (effects (font (size 1.27 1.27)))
-    )
-    (property "Value" "KEYBOARD" (at 386.08 139.0396 0)
-      (effects (font (size 1.27 1.27)))
-    )
-    (property "Footprint" "Connector_PinHeader_2.54mm:PinHeader_2x08_P2.54mm_Vertical" (at 384.81 149.86 0)
-      (effects (font (size 1.27 1.27)) hide)
-    )
-    (property "Datasheet" "~" (at 384.81 149.86 0)
-      (effects (font (size 1.27 1.27)) hide)
-    )
-    (pin "1")
-    (pin "10")
-    (pin "11")
-    (pin "12")
-    (pin "13")
-    (pin "14")
-    (pin "15")
-    (pin "16")
-    (pin "2")
-    (pin "3")
-    (pin "4")
-    (pin "5")
-    (pin "6")
-    (pin "7")
-    (pin "8")
-    (pin "9")
-    (instances
-      (project "we816mark2"
-        (path "/ca9b74ce-0dee-401c-9544-f599f4cf538d/00000000-0000-0000-0000-00005ffce1f8"
-          (reference "J3") (unit 1)
-        )
-      )
-    )
-  )
   (symbol (lib_id "power:GND") (at 393.7 160.02 0) (unit 1)
     (in_bom yes) (on_board yes) (dnp no)
@@
     )
   )
+  (symbol (lib_id "Connector_Generic:Conn_02x08_Odd_Even") (at 384.81 149.86 0) (unit 1)
+    (in_bom yes) (on_board yes) (dnp no) (fields_autoplaced)
+    (property "Reference" "J3" (at 386.08 137.16 0)
+      (effects (font (size 1.27 1.27)))
+    )
+    (property "Value" "Keyboard" (at 386.08 139.7 0)
+      (effects (font (size 1.27 1.27)))
+    )
+    (property "Footprint" "Connector_PinHeader_2.54mm:PinHeader_2x08_P2.54mm_Vertical" (at 384.81 149.86 0)
+      (effects (font (size 1.27 1.27)) hide)
+    )
+    (property "Datasheet" "~" (at 384.81 149.86 0)
+      (effects (font (size 1.27 1.27)) hide)
+    )
+    (pin "1")
+    (pin "10")
+    (pin "11")
+    (pin "12")
+    (pin "13")
+    (pin "14")
+    (pin "15")
+    (pin "16")
+    (pin "2")
+    (pin "3")
+    (pin "4")
+    (pin "5")
+    (pin "6")
+    (pin "7")
+    (pin "8")
+    (pin "9")
+    (instances
+      (project "we816mark2"
+        (path "/ca9b74ce-0dee-401c-9544-f599f4cf538d/00000000-0000-0000-0000-00005ffce1f8"
+          (reference "J3") (unit 1)
+        )
+      )
+    )
+  )
   (symbol (lib_id "Power_Management:DS1210") (at 185.42 123.19 0) (unit 1)
     (in_bom yes) (on_board yes) (dnp no)
@@
         )
       )
+    )
+  )
+  (symbol (lib_id "Oscillator:CXO_DIP14") (at 49.53 254 0) (unit 1)
+    (in_bom yes) (on_board yes) (dnp no)
+    (property "Reference" "X1" (at 60.96 250.8759 0)
+      (effects (font (size 1.27 1.27)))
+    )
+    (property "Value" "CXO_DIP14" (at 55.88 246.38 0)
+      (effects (font (size 1.27 1.27)))
+    )
+    (property "Footprint" "Oscillator:Oscillator_DIP-14" (at 60.96 262.89 0)
+      (effects (font (size 1.27 1.27)) hide)
+    )
+    (property "Datasheet" "http://cdn-reichelt.de/documents/datenblatt/B400/OSZI.pdf" (at 46.99 254 0)
+      (effects (font (size 1.27 1.27)) hide)
+    )
+    (pin "1")
+    (pin "14")
+    (pin "7")
+    (pin "8")
+    (instances
+      (project "we816mark2"
+        (path "/ca9b74ce-0dee-401c-9544-f599f4cf538d/00000000-0000-0000-0000-00005ffce1f8"
+          (reference "X1") (unit 1)
+        )
+      )

Commit message: rtc updates
Parts:
- removed BT1: Battery_Cell, CUSTOMLibrary:Battery_Holder_Coin_2032_BS-7_FIXED, symbol Device:Battery_Cell
- removed C21 (x2): 33 pF, Capacitor_THT:C_Rect_L7.0mm_W2.0mm_P5.00mm, symbol Device:C_Small
- removed C34: 30 pF, Capacitor_THT:CP_Radial_D4.0mm_P2.00mm, symbol Device:C_Trim_Small
- removed JP1, JP2: BYPASS, Connector_PinHeader_2.54mm:PinHeader_1x02_P2.54mm_Vertical, symbol Jumper:Jumper_2_Open
- removed K4: VCC TOL 0, Connector_PinHeader_2.54mm:PinHeader_1x03_P2.54mm_Vertical, symbol Connector_Generic:Conn_01x03
- removed R16 (x3): 100kΩ, Resistor_THT:R_Axial_DIN0204_L3.6mm_D1.6mm_P5.08mm_Horizontal, symbol Device:R_Small
- removed U7: RP5C01, Package_DIP:DIP-18_W7.62mm_Socket_LongPads, symbol RPi_pico:rp5c01
- removed U8: 74LS175, Package_DIP:DIP-16_W7.62mm_Socket_LongPads, symbol 74xx:74LS175
- removed U9: DS1210, Package_DIP:DIP-8_W7.62mm_Socket_LongPads, symbol Power_Management:DS1210
- added BT2: Battery_Cell, CUSTOMLibrary:Battery_Holder_Coin_2032_BS-7_FIXED, symbol Device:Battery_Cell
- added U19: DS1501WN, Package_DIP:DIP-28_W15.24mm_Socket_LongPads, symbol RPi_pico:DS1501WN
Connections:
- net A0: now also U19.10 (A0)
- net A1: now also U19.9 (A1)
- net A2: now also U19.8 (A2)
- net A3: now also U19.7 (A3)
- net D0: now also U19.11 (DQ0)
- net D1: now also U19.12 (DQ1)
- net D2: now also U19.13 (DQ2)
- net D3: now also U19.15 (DQ3)
- net D4: now also U19.16 (DQ4)
- net D5: now also U19.17 (DQ5)
- net D6: now also U19.18 (DQ6)
- net D7: now also U19.19 (DQ7)
- net GND: now also BT2.2 (-), U19.14 (GND_2), U19.21 (GND), U19.24 (*KS), U19.26 (VBAUX)
- net RD: now also U19.22 (OE)
- net USERCA_2: now also U19.5 (*IRQ)
- net VCC: now also U19.28 (VCC)
- net WR: now also U19.27 (*WE)
- net ~{RTC_CS}: now also U19.20 (*CE)
- net at X3.1: now also U19.2 (X1)
- net at X3.2: now also U19.3 (X2)
- new net: BT2.1 (+), U19.25 (VBAT)
- new net A4: U19.6 (A4)
- no-connect marks 24 -> 23
Other:
- note removed: "JP1 AND JP3 U2 DS1210 INSTALLED CLOSE BOTH TO BYPASS DEFAULT BOTH OPEN"
- note removed: "NOTE: K1 VCC TOLERANCE 1-2 CLOSED 10% 2-3 CLOSED 5%"
- moved on the sheet: X3
