File: Hardware/file60340596.kicad_sch (KiCad schematic)
At the start: 4 parts, among them K1 1&2 FOR SMALL ROM, 2&3 FOR LA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, U12 GAL16V8, U13 GAL20V8, U14 GAL16V8

Commit message: mark 2 work
Parts:
- added U6: GAL16V8, Package_DIP:DIP-20_W7.62mm_Socket_LongPads, symbol Logic_Programmable:GAL16V8
- K1: symbol Connector:Conn_01x03_Male -> Connector:Conn_01x03_Pin
Connections:
- net A15: now also U6.1 (I1/CLK)
- net A16: now also U6.2 (I2)
- net A17: now also U6.3 (I3)
- net A18: now also U6.4 (I4)
- net A19: now also U6.5 (I5)
- net A20: now also U6.6 (I6)
- net A21: now also U6.7 (I7)
- net A22: now also U6.8 (I8)
- net A23: now also U6.9 (I9)
- net GND: now also U6.10 (GND)
- net VCC: now also U6.20 (VCC)
- net WR: now also U12.11 (I10/~{OE})
- net ~{RTC_CS}: now reaches U12.16 (IO4)
- net ~{RTC_AD_WR}: now reaches U12.18 (IO2)
- new net VIDEO_WINDOW: U6.19 (IO1)
- no-connect marks 11 -> 16

Commit message: pcb work
Other:
- title: (none) -> WE65816 - MARK2
Changed lines of the file:
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@@
 (kicad_sch (version 20230121) (generator eeschema)
   (paper "B")
+  (title_block
+    (title "WE65816 - MARK2")
+    (rev "V0.80")
+  )
   (no_connect (at 91.44 201.93))
   (no_connect (at 91.44 199.39))

Commit message: initial pico firmware
Parts:
- removed U13: GAL20V8, Package_DIP:DIP-24_W7.62mm_Socket_LongPads, symbol Logic_Programmable:PAL20L8
- added U13: ATF22V10, Package_DIP:DIP-24_W7.62mm_Socket_LongPads, symbol RPi_pico:ATF22V11
Connections:
- net A10: now also U13.2 (I2)
- net A11: now also U13.3 (I3)
- net A12: now also U13.4 (I4/PD)
- net A13: now also U13.5 (I5)
- net A14: now also U13.6 (I6)
- net A15: now also U13.7 (I7)
- net A16: now also U13.8 (I8)
- net A17: now also U13.9 (I9)
- net A18: now also U13.10 (I10)
- net A19: now also U13.11 (I11)
- net A20: now also U13.14 (IO14)
- net A21: now also U13.1 (CLK/I1)
- net A22: now also U13.13 (I13)
- net A23: now also U13.23 (IO23)
- net A8: now also U13.21 (IO21)
- net A9: now also U13.22 (IO22)
- net BUS: now also U13.18 (IO18)
- net CS_RAM: now also U13.16 (IO16)
- net CS_ROM: now also U13.15 (IO15)
- net GND: now also U13.12 (GND)
- net IO: now also U13.17 (IO17)
- net O1_ROM: now also U13.19 (IO19)
- net VCC: now also U13.24 (VCC)
- net at K1.2 (Pin_2): now also U13.20 (I020)
Other:
- moved on the sheet: K1

Commit message: graphics work
Parts:
- added U16: GAL16V8, Package_DIP:DIP-20_W7.62mm_Socket_LongPads, symbol Logic_Programmable:GAL16V8
Connections:
- net CLK_CPU: now also U16.1 (I1/CLK)
- net CS_ROM: now also U16.6 (I6)
- net GND: now also U16.10 (GND), U16.11 (I10/~{OE})
- net IO: now also U16.7 (I7)
- net RW: now also U16.4 (I4)
- net VCC: now also U16.20 (VCC)
- net VDA: now also U16.2 (I2)
- net VPA: now also U16.3 (I3)
- net VIDEO_WS: now reaches U6.18 (IO2)
- net VIDEO_WS: now also U16.5 (I5)
- new net FF1: U16.12 (IO8)
- new net FF2: U16.13 (IO7)
- new net RESET: U16.9 (I9)
- new net WAIT: U16.14 (IO6)
- new net WS1: U16.15 (IO5)
- new net WS2: U16.16 (IO4)
- no-connect marks 16 -> 19
Other:
- note added: "System can be ran with Wait State Generator (U16) out of system Video and IO are 2 wait states ROM is 1 wait state"

Commit message: BASIC work
Parts:
- removed K1: 1&2 FOR SMALL ROM, 2&3 FOR LARGE ROM, Connector_PinHeader_2.54mm:PinHeader_1x03_P2.54mm_Vertical, symbol Connector:Conn_01x03_Pin
Connections:
- no-connect marks 19 -> 20
Changed lines of the file:
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@@
   (no_connect (at 116.84 179.07))
   (no_connect (at 116.84 181.61))
+  (no_connect (at 118.11 134.62))
   (no_connect (at 116.84 95.25))
   (no_connect (at 213.36 87.63))
@@
     (stroke (width 0) (type default))
   )
-  (wire (pts (xy 118.11 134.62) (xy 147.32 134.62))
-    (stroke (width 0) (type default))
-  )
   (wire (pts (xy 86.36 77.47) (xy 91.44 77.47))
     (stroke (width 0) (type default))
@@
     (stroke (width 0) (type default))
   )
-  (wire (pts (xy 147.32 137.16) (xy 147.32 139.7))
-    (stroke (width 0) (type default))
-  )
   (wire (pts (xy 182.88 179.07) (xy 187.96 179.07))
     (stroke (width 0) (type default))
@@
   )
   (wire (pts (xy 86.36 82.55) (xy 91.44 82.55))
-    (stroke (width 0) (type default))
-  )
-  (wire (pts (xy 147.32 125.73) (xy 147.32 132.08))
     (stroke (width 0) (type default))
   )
@@
     )
   )
-  (symbol (lib_id "Connector:Conn_01x03_Pin") (at 152.4 134.62 0) (mirror y) (unit 1)
-    (in_bom yes) (on_board yes) (dnp no)
-    (property "Reference" "K1" (at 153.67 134.62 90)
-      (effects (font (size 1.27 1.27)))
-    )
-    (property "Value" "1&2 FOR SMALL ROM, 2&3 FOR LARGE ROM " (at 173.99 133.35 0)
-      (effects (font (size 1.016 1.016)))
-    )
-    (property "Footprint" "Connector_PinHeader_2.54mm:PinHeader_1x03_P2.54mm_Vertical" (at 152.4 134.62 0)
-      (effects (font (size 1.27 1.27)) hide)
-    )
-    (property "Datasheet" "~" (at 152.4 134.62 0)
-      (effects (font (size 1.27 1.27)) hide)
-    )
-    (pin "1")
-    (pin "2")
-    (pin "3")
-    (instances
-      (project "we816mark2"
-        (path "/ca9b74ce-0dee-401c-9544-f599f4cf538d/00000000-0000-0000-0000-000060340597"
-          (reference "K1") (unit 1)
-        )
-      )
-    )
-  )
-  (symbol (lib_id "power:VCC") (at 147.32 125.73 0) (unit 1)
-    (in_bom yes) (on_board yes) (dnp no)
-    (property "Reference" "#PWR028" (at 147.32 129.54 0)
-      (effects (font (size 1.27 1.27)) hide)
-    )
-    (property "Value" "VCC" (at 147.701 121.3358 0)
-      (effects (font (size 1.27 1.27)))
-    )
-    (property "Footprint" "" (at 147.32 125.73 0)
-      (effects (font (size 1.27 1.27)) hide)
-    )
-    (property "Datasheet" "" (at 147.32 125.73 0)
-      (effects (font (size 1.27 1.27)) hide)
-    )
-    (pin "1")
-    (instances
-      (project "we816mark2"
-        (path "/ca9b74ce-0dee-401c-9544-f599f4cf538d/00000000-0000-0000-0000-000060340597"
-          (reference "#PWR028") (unit 1)
-        )
-      )
-    )
-  )
-  (symbol (lib_id "power:GND") (at 147.32 139.7 0) (unit 1)
-    (in_bom yes) (on_board yes) (dnp no)
-    (property "Reference" "#PWR029" (at 147.32 146.05 0)
-      (effects (font (size 1.27 1.27)) hide)
-    )
-    (property "Value" "GND" (at 147.447 144.0942 0)
-      (effects (font (size 1.27 1.27)))
-    )
-    (property "Footprint" "" (at 147.32 139.7 0)
-      (effects (font (size 1.27 1.27)) hide)
-    )
-    (property "Datasheet" "" (at 147.32 139.7 0)
-      (effects (font (size 1.27 1.27)) hide)
-    )
-    (pin "1")
-    (instances
-      (project "we816mark2"
-        (path "/ca9b74ce-0dee-401c-9544-f599f4cf538d/00000000-0000-0000-0000-000060340597"
-          (reference "#PWR029") (unit 1)
-        )
-      )
-    )
-  )

Commit message: rtc updates
Connections:
- net VDA: now also U12.12 (IO8)
- no-connect marks 20 -> 19
Changed lines of the file:
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@@
   (title_block
     (title "WE65816 - MARK2")
-    (date "2024-08-11")
+    (date "2024-09-07")
     (rev "V0.90")
   )
@@
   (no_connect (at 116.84 181.61))
   (no_connect (at 118.11 134.62))
-  (no_connect (at 116.84 95.25))
   (no_connect (at 213.36 87.63))
   (no_connect (at 213.36 90.17))
@@
     (stroke (width 0) (type default))
   )
+  (wire (pts (xy 116.84 95.25) (xy 120.65 95.25))
+    (stroke (width 0) (type default))
+  )
   (wire (pts (xy 116.84 90.17) (xy 120.65 90.17))
     (stroke (width 0) (type default))
@@
       (effects (font (size 1.27 1.27)) (justify left) hide)
     )
+  )
+  (global_label "VDA" (shape input) (at 120.65 95.25 0) (fields_autoplaced)
+    (effects (font (size 1.524 1.524)) (justify left))
+    (property "Intersheetrefs" "${INTERSHEET_REFS}" (at 127.488 95.25 0)
+      (effects (font (size 1.27 1.27)) (justify left) hide)
+    )

Commit message: add basic RTC functions
Parts:
- removed U16: GAL16V8, Package_DIP:DIP-20_W7.62mm_Socket_LongPads, symbol Logic_Programmable:GAL16V8
Connections:
- net VIDEO_WS: no longer names the net of U6.18 (IO2)
- net ~{RTC_AD_WR}: no longer names the net of U12.18 (IO2)
- no-connect marks 19 -> 17
Other:
- note removed: "System can be ran with Wait State Generator (U16) out of system Video and IO are 2 wait states ROM is 1 wait state"
