File: Hardware/file60341279.kicad_sch (KiCad schematic)
At the start: 11 parts, among them J6 INTERRUPT SELECT, J7 expansion port, U20 74LS245, U21 74LS244, U22 74LS245, U23 74LS245, U24 74LS245, U3 74LS06N, U4 74LS14

Commit message: mark 2 work
Parts:
- J6: symbol Connector_Generic:Conn_02x04_Counter_Clockwise -> Connector_Generic:Conn_02x03_Counter_Clockwise
Connections:
- net V_INT is gone; now on net B_INT: J6.4 (Pin_4)
- net B_INT: no longer J6.7 (Pin_7), J6.8 (Pin_8)

Commit message: pcb work
Other:
- title: (none) -> WE65816 - MARK2
Changed lines of the file:
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@@
 (kicad_sch (version 20230121) (generator eeschema)
   (paper "B")
+  (title_block
+    (title "WE65816 - MARK2")
+    (rev "V0.80")
+  )
   (junction (at 104.14 39.37) (diameter 0) (color 0 0 0 0)
   )

Commit message: graphics work
Parts:
- U3: footprint Package_DIP:DIP-14_W7.62mm_Socket -> Package_DIP:DIP-14_W7.62mm_Socket_LongPads
Changed lines of the file:
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@@
   (title_block
     (title "WE65816 - MARK2")
+    (date "2024-08-11")
     (rev "V0.90")
   )
@@
       (effects (font (size 1.27 1.27)) (justify left bottom))
     )
-    (property "Footprint" "Package_DIP:DIP-14_W7.62mm_Socket" (at 72.39 71.12 0)
+    (property "Footprint" "Package_DIP:DIP-14_W7.62mm_Socket_LongPads" (at 72.39 71.12 0)
       (effects (font (size 1.27 1.27)) hide)
     )
@@
       (effects (font (size 1.27 1.27)) (justify left bottom))
     )
-    (property "Footprint" "Package_DIP:DIP-14_W7.62mm_Socket" (at 57.15 39.37 0)
+    (property "Footprint" "Package_DIP:DIP-14_W7.62mm_Socket_LongPads" (at 57.15 39.37 0)
       (effects (font (size 1.27 1.27)) hide)
     )
@@
       (effects (font (size 1.27 1.27)) (justify left bottom))
     )
-    (property "Footprint" "Package_DIP:DIP-14_W7.62mm_Socket" (at 110.49 26.67 0)
-      (effects (font (size 1.27 1.27)) hide)
-    )
+    (property "Footprint" "Package_DIP:DIP-14_W7.62mm_Socket_LongPads" (at 110.49 26.67 0)
+      (effects (font (size 1.27 1.27)) hide)
+    )

Commit message: BASIC graphics work
Parts:
- J7: value expansion port -> Expansion Port
