File: Hardware/we816mark2.kicad_sch (KiCad schematic)
At the start: 43 parts, among them U10 74AC04, U2 7406, U3 74LS06N, U35 LM3940, U4 74LS14

Commit message: pcb work
Other:
- title: (none) -> WE65816 - MARK2
Changed lines of the file:
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@@
   (paper "B")
   (title_block
-    (date "23 jan 2013")
+    (title "WE65816 - MARK2")
+    (rev "V0.80")
   )
   (junction (at 196.85 241.3) (diameter 0) (color 0 0 0 0)

Commit message: graphics work
Parts:
- U2, U3: footprint Package_DIP:DIP-14_W7.62mm_Socket -> Package_DIP:DIP-14_W7.62mm_Socket_LongPads
Changed lines of the file:
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@@
   (title_block
     (title "WE65816 - MARK2")
+    (date "2024-08-11")
     (rev "V0.90")
   )
@@
       (effects (font (size 1.27 1.27)) (justify left bottom))
     )
-    (property "Footprint" "Package_DIP:DIP-14_W7.62mm_Socket" (at 360.68 124.46 0)
+    (property "Footprint" "Package_DIP:DIP-14_W7.62mm_Socket_LongPads" (at 360.68 124.46 0)
       (effects (font (size 1.27 1.27)) hide)
     )
@@
       (effects (font (size 1.27 1.27)) (justify left bottom))
     )
-    (property "Footprint" "Package_DIP:DIP-14_W7.62mm_Socket" (at 360.68 162.56 0)
+    (property "Footprint" "Package_DIP:DIP-14_W7.62mm_Socket_LongPads" (at 360.68 162.56 0)
       (effects (font (size 1.27 1.27)) hide)
     )
@@
       (effects (font (size 1.27 1.27)))
     )
-    (property "Footprint" "Package_DIP:DIP-14_W7.62mm_Socket" (at 320.04 125.73 0)
+    (property "Footprint" "Package_DIP:DIP-14_W7.62mm_Socket_LongPads" (at 320.04 125.73 0)
       (effects (font (size 1.27 1.27)) hide)
     )
@@
       (effects (font (size 1.27 1.27)))
     )
-    (property "Footprint" "Package_DIP:DIP-14_W7.62mm_Socket" (at 320.04 135.89 0)
+    (property "Footprint" "Package_DIP:DIP-14_W7.62mm_Socket_LongPads" (at 320.04 135.89 0)
       (effects (font (size 1.27 1.27)) hide)
     )
@@
       (effects (font (size 1.27 1.27)))
     )
-    (property "Footprint" "Package_DIP:DIP-14_W7.62mm_Socket" (at 320.04 146.05 0)
+    (property "Footprint" "Package_DIP:DIP-14_W7.62mm_Socket_LongPads" (at 320.04 146.05 0)
       (effects (font (size 1.27 1.27)) hide)
     )
@@
       (effects (font (size 1.27 1.27)) (justify left bottom))
     )
-    (property "Footprint" "Package_DIP:DIP-14_W7.62mm_Socket" (at 360.68 189.23 0)
+    (property "Footprint" "Package_DIP:DIP-14_W7.62mm_Socket_LongPads" (at 360.68 189.23 0)
       (effects (font (size 1.27 1.27)) hide)
     )
@@
       (effects (font (size 1.27 1.27)))
     )
-    (property "Footprint" "Package_DIP:DIP-14_W7.62mm_Socket" (at 363.22 87.63 0)
+    (property "Footprint" "Package_DIP:DIP-14_W7.62mm_Socket_LongPads" (at 363.22 87.63 0)
       (effects (font (size 1.27 1.27)) hide)
     )
@@
       (effects (font (size 1.27 1.27)) (justify left bottom))
     )
-    (property "Footprint" "Package_DIP:DIP-14_W7.62mm_Socket" (at 347.98 87.63 0)
-      (effects (font (size 1.27 1.27)) hide)
-    )
+    (property "Footprint" "Package_DIP:DIP-14_W7.62mm_Socket_LongPads" (at 347.98 87.63 0)
+      (effects (font (size 1.27 1.27)) hide)
+    )
